File: kicad/release-modem-atmega328p/design.kicad_pcb (KiCad board)
At the start: 2 copper layers, 23 x 15.4 mm, 23 parts, among them J1 ADC-Debug, J3 UART0, U3 ATmega328P-AU, Y1 AB308-16.000MHZ

Commit message: Rework the piezo input to use an OPA1641 opamp
Parts:
- removed D1, D3: 1N4007, custom:WP_D_SOD-123
- removed J1: ADC-Debug, Connector_PinHeader_2.54mm:PinHeader_1x01_P2.54mm_Vertical
- added ADC1: ADC-Debug, custom:WP_PinSocket_1x02_P2.54mm_Vertical, F.Cu at (134.0, 62.2)
- added BAS4004: BAS40-04, Package_TO_SOT_SMD:SOT-23, B.Cu at (144.8, 58.9)
- added C1: 22uF, custom:WP_C_0805_2012Metric_Pad1.15x1.40mm_HandSolder, B.Cu at (135.4, 59.6)
- added C2: 0.1uF, custom:WP_C_0805_2012Metric_Pad1.15x1.40mm_HandSolder, F.Cu at (132.6, 59.2)
- added C3: 22uF, custom:WP_C_0805_2012Metric_Pad1.15x1.40mm_HandSolder, F.Cu at (137.8, 64.5)
- added EN1: LineInJumper, Jumper:SolderJumper-2_P1.3mm_Open_Pad1.0x1.5mm, F.Cu at (141.6, 64.8)
- added LINE1: LineIn, custom:WP_PinSocket_1x02_P2.54mm_Vertical, F.Cu at (138.7, 61.9)
- added OPA1641: OPA1641AQDGKRQ1, Package_SO:VSSOP-8_3.0x3.0mm_P0.65mm, F.Cu at (144.8, 62.9)
- added R10: 1M, custom:WP_R_0805_2012Metric_Pad1.15x1.40mm_HandSolder, B.Cu at (145.2, 66.8)
- added R12: 1K, custom:WP_R_0805_2012Metric_Pad1.15x1.40mm_HandSolder, F.Cu at (145.2, 68.8)
- added R13: 1K, custom:WP_R_0805_2012Metric_Pad1.15x1.40mm_HandSolder, B.Cu at (142.6, 65.4)
- R5, R7: moved to B.Cu
- R6: value 10K -> 47K
- R9: value 1M -> 47K; moved to F.Cu
- moved PIEZO1 10.7 mm to (143.1, 70.5), turned to 180 degrees
- moved R6 6.21 mm to (135.4, 59.4), turned to 180 degrees
- moved R8 5.74 mm to (144.0, 63.0), turned to 0 degrees
- moved R9 5.36 mm to (139.1, 59.4), turned to 180 degrees
- moved R7 4.27 mm to (132.0, 61.5), turned to 90 degrees
- moved R5 3.42 mm to (136.0, 63.5)
- moved AVRISP6 1.14 mm to (140.0, 68.1)
Connections:
- PIEZO1 pad 1: Net-(PIEZO1-Pad1) -> GND
- PIEZO1 pad 2: ADC0 -> Net-(PIEZO1-Pad2)
- R5 pad 1: Net-(D1-Pad2) -> GND
- R5 pad 2: Net-(PIEZO1-Pad1) -> ADC0
- R6 pad 1: Net-(D3-Pad1) -> Vmid
- R6 pad 2: Net-(PIEZO1-Pad1) -> 5V-In
- R7 pad 1: 5V-In -> ADC0
- R7 pad 2: Net-(D1-Pad2) -> 5V-In
- R8 pad 1: GND -> Net-(EN1-Pad1)
- R8 pad 2: Net-(D3-Pad1) -> Net-(OPA1641-Pad2)
- R9 pad 1: ADC0 -> GND
- R9 pad 2: Net-(PIEZO1-Pad1) -> Vmid
Routing:
- net GND: track 144.0 -> 173.6 mm, vias 5 -> 6
- net Vmid: track 0.00 -> 17.6 mm, vias 0 -> 2
- net Net-(D3-Pad1): track 17.4 -> 0.00 mm, vias 1 -> 0
- net 5V-In: track 60.9 -> 77.8 mm, vias 1 -> 3
- net Net-(BAS4004-Pad3): track 0.00 -> 14.9 mm, vias 0 -> 1
- net Net-(OPA1641-Pad2): track 0.00 -> 12.5 mm, vias 0 -> 1
- net Net-(PIEZO1-Pad1): track 6.71 -> 0.00 mm
- net Net-(D1-Pad2): track 6.03 -> 0.00 mm
- net Net-(EN1-Pad1): track 0.00 -> 6.01 mm, vias 0 -> 1
- net Net-(C3-Pad2): track 0.00 -> 5.24 mm
- net Net-(PIEZO1-Pad2): track 0.00 -> 4.17 mm
- net ADC0: track 12.8 -> 11.0 mm
- net RESET: track 18.9 -> 20.2 mm
- net Net-(AVRISP6-Pad4): track 8.74 -> 9.88 mm
- net Net-(AVRISP6-Pad1): track 9.98 -> 11.1 mm
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Other:
- board size 23 x 15.4 mm -> 28.8 x 15.4 mm
- board text added: "2025-04-16 V3"
- board text added: "HydroModem(Piezo) + OPA1641"
- board text added: "LINE"
- board text removed: "2025-03-15 V1"
